File: pcb/node.brd (EAGLE design)
At the start: 25 x 25 mm, 10 parts, among them J1 AVR_SPI_PRG_62X3_LOCK

Commit message: placing parts
Parts:
- added C1: 100u, rcl:SANYO-OSCON_SMD_C6
- added C2: 4u7, rcl:E5-5
- moved U$1 8.13 mm to (17.8, 20.3), turned to 90 degrees
- moved U$3 3.59 mm to (8.89, 16.5)
Connections:
- net GND: now also C1.-, C2.-
- net VBATT: now also C2.+
- net VCC: now also C1.+
Changed lines of the file:
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@@
 </autorouter>
 <elements>
-<element name="U$1" library="SparkFun-DigitalIC" package="SO08" value="ATTINY13SOIC" x="12.7" y="13.97"/>
+<element name="U$1" library="SparkFun-DigitalIC" package="SO08" value="ATTINY13SOIC" x="17.78" y="20.32" rot="R90"/>
 <element name="U$2" library="ukhas" package="SOT23-6" value="MCP1640" x="16.51" y="3.81" rot="R180"/>
-<element name="U$3" library="jonsowman" package="SOT23-5L" value="BU49X_VDET_SOT235" x="6.35" y="13.97"/>
+<element name="U$3" library="jonsowman" package="SOT23-5L" value="BU49X_VDET_SOT235" x="8.89" y="16.51"/>
 <element name="DF" library="jonsowman" package="BOURNS_SRN5040_L" value="4u7" x="21.59" y="3.81" rot="R90"/>
 <element name="J1" library="SparkFun-Connectors" package="2X3_LOCK" value="AVR_SPI_PRG_62X3_LOCK" x="7.62" y="2.54"/>
@@
 <element name="U$4" library="hoperf" package="RFM" value="RFM69HW" x="23.495" y="24.13" rot="R180"/>
 <element name="JP1" library="SparkFun-Connectors" package="1X01" value="M01PTH" x="1.27" y="21.59"/>
+<element name="C1" library="rcl" package="SANYO-OSCON_SMD_C6" value="100u" x="17.78" y="11.43"/>
+<element name="C2" library="rcl" package="E5-5" value="4u7" x="-6.35" y="13.97"/>
 </elements>
 <signals>
@@
 <contactref element="U$4" pad="GNDB"/>
 <contactref element="U$4" pad="GNDA"/>
+<contactref element="C1" pad="-"/>
+<contactref element="C2" pad="-"/>
+<wire x1="14.98" y1="11.43" x2="20.3962" y2="22.225" width="0" layer="19" extent="1-1"/>
+<wire x1="13.12" y1="7.62" x2="14.98" y2="11.43" width="0" layer="19" extent="1-1"/>
+<wire x1="12.7" y1="5.08" x2="13.12" y2="7.62" width="0" layer="19" extent="1-1"/>
+<wire x1="16.51" y1="4.96" x2="12.7" y2="5.08" width="0" layer="19" extent="1-1"/>
+<wire x1="9.84" y1="15.21" x2="14.98" y2="11.43" width="0" layer="19" extent="1-1"/>
+<wire x1="3.84375" y1="19.24125" x2="9.84" y2="15.21" width="0" layer="19" extent="1-1"/>
 <wire x1="3.84375" y1="23.0825" x2="3.84375" y2="19.24125" width="0" layer="19" extent="1-1"/>
-<wire x1="16.51" y1="4.96" x2="3.84375" y2="23.0825" width="0" layer="19" extent="1-1"/>
-<wire x1="12.7" y1="5.08" x2="16.51" y2="4.96" width="0" layer="19" extent="1-1"/>
-<wire x1="13.12" y1="7.62" x2="12.7" y2="5.08" width="0" layer="19" extent="1-1"/>
-<wire x1="14.605" y1="11.3538" x2="13.12" y2="7.62" width="0" layer="19" extent="1-1"/>
-<wire x1="7.3" y1="12.67" x2="14.605" y2="11.3538" width="0" layer="19" extent="1-1"/>
-<wire x1="2.54" y1="4.81" x2="7.3" y2="12.67" width="0" layer="19" extent="1-1"/>
+<wire x1="2.54" y1="4.81" x2="12.7" y2="5.08" width="0" layer="19" extent="1-1"/>
+<wire x1="-3.81" y1="13.97" x2="2.54" y2="4.81" width="0" layer="19" extent="1-1"/>
 </signal>
 <signal name="VCC">
@@
 <contactref element="J1" pad="2"/>
 <contactref element="U$4" pad="VCC"/>
-<wire x1="6.35" y1="12.67" x2="10.795" y2="16.5862" width="0" layer="19" extent="1-1"/>
-<wire x1="23.495" y1="23.0825" x2="6.35" y2="12.67" width="0" layer="19" extent="1-1"/>
-<wire x1="7.62" y1="5.08" x2="23.495" y2="23.0825" width="0" layer="19" extent="1-1"/>
-<wire x1="16.51" y1="2.66" x2="7.62" y2="5.08" width="0" layer="19" extent="1-1"/>
-<wire x1="18.63" y1="7.62" x2="16.51" y2="2.66" width="0" layer="19" extent="1-1"/>
+<contactref element="C1" pad="+"/>
+<wire x1="15.1638" y1="18.415" x2="23.495" y2="23.0825" width="0" layer="19" extent="1-1"/>
+<wire x1="8.89" y1="15.21" x2="15.1638" y2="18.415" width="0" layer="19" extent="1-1"/>
+<wire x1="20.58" y1="11.43" x2="15.1638" y2="18.415" width="0" layer="19" extent="1-1"/>
+<wire x1="18.63" y1="7.62" x2="20.58" y2="11.43" width="0" layer="19" extent="1-1"/>
+<wire x1="16.51" y1="2.66" x2="18.63" y2="7.62" width="0" layer="19" extent="1-1"/>
+<wire x1="7.62" y1="5.08" x2="16.51" y2="2.66" width="0" layer="19" extent="1-1"/>
 </signal>
 <signal name="N$1">
@@
 <contactref element="U$1" pad="6"/>
 <contactref element="U$4" pad="MISO"/>
-<wire x1="13.335" y1="16.5862" x2="3.84375" y2="15.0825" width="0" layer="19" extent="1-1"/>
-<wire x1="7.62" y1="2.54" x2="13.335" y2="16.5862" width="0" layer="19" extent="1-1"/>
+<wire x1="3.84375" y1="15.0825" x2="15.1638" y2="20.955" width="0" layer="19" extent="1-1"/>
+<wire x1="7.62" y1="2.54" x2="3.84375" y2="15.0825" width="0" layer="19" extent="1-1"/>
 </signal>
 <signal name="RESET">
 <contactref element="J1" pad="5"/>
 <contactref element="U$1" pad="1"/>
-<wire x1="12.7" y1="2.54" x2="10.795" y2="11.3538" width="0" layer="19" extent="1-1"/>
+<wire x1="12.7" y1="2.54" x2="20.3962" y2="18.415" width="0" layer="19" extent="1-1"/>
 </signal>
 <signal name="MOSI">
@@
 <contactref element="U$1" pad="5"/>
 <contactref element="U$4" pad="MOSI"/>
-<wire x1="14.605" y1="16.5862" x2="3.84375" y2="13.0825" width="0" layer="19" extent="1-1"/>
-<wire x1="10.16" y1="4.826" x2="14.605" y2="16.5862" width="0" layer="19" extent="1-1"/>
+<wire x1="3.84375" y1="13.0825" x2="15.1638" y2="22.225" width="0" layer="19" extent="1-1"/>
+<wire x1="10.16" y1="4.826" x2="3.84375" y2="13.0825" width="0" layer="19" extent="1-1"/>
 </signal>
 <signal name="N$4">
 <contactref element="U$1" pad="2"/>
 <contactref element="U$2" pad="3"/>
-<wire x1="15.56" y1="4.96" x2="12.065" y2="11.3538" width="0" layer="19" extent="1-1"/>
+<wire x1="15.56" y1="4.96" x2="20.3962" y2="19.685" width="0" layer="19" extent="1-1"/>
 </signal>
 <signal name="DET/SCK">
@@
 <contactref element="J1" pad="3"/>
 <contactref element="U$4" pad="SCK"/>
-<wire x1="12.065" y1="16.5862" x2="3.84375" y2="17.0825" width="0" layer="19" extent="1-1"/>
-<wire x1="5.4" y1="12.67" x2="12.065" y2="16.5862" width="0" layer="19" extent="1-1"/>
-<wire x1="10.16" y1="2.286" x2="5.4" y2="12.67" width="0" layer="19" extent="1-1"/>
+<wire x1="7.94" y1="15.21" x2="15.1638" y2="19.685" width="0" layer="19" extent="1-1"/>
+<wire x1="3.84375" y1="17.0825" x2="7.94" y2="15.21" width="0" layer="19" extent="1-1"/>
+<wire x1="10.16" y1="2.286" x2="7.94" y2="15.21" width="0" layer="19" extent="1-1"/>
 </signal>
 <signal name="N$2">
@@
 <contactref element="DF" pad="P$1"/>
 <contactref element="U$2" pad="6"/>
+<contactref element="C2" pad="+"/>
 <wire x1="17.46" y1="2.66" x2="21.59" y2="2.01" width="0" layer="19" extent="1-1"/>
 <wire x1="2.54" y1="2.81" x2="17.46" y2="2.66" width="0" layer="19" extent="1-1"/>
+<wire x1="-8.89" y1="13.97" x2="2.54" y2="2.81" width="0" layer="19" extent="1-1"/>
 </signal>
 <signal name="RFM_SS">
 <contactref element="U$4" pad="NSS"/>
 <contactref element="U$1" pad="3"/>
-<wire x1="13.335" y1="11.3538" x2="3.84375" y2="10.92375" width="0" layer="19" extent="1-1"/>
+<wire x1="3.84375" y1="10.92375" x2="20.3962" y2="20.955" width="0" layer="19" extent="1-1"/>
 </signal>
 <signal name="N$3">

Commit message: routing commence
Parts:
- added D1: (no value), dtb:SOD123
- added R3: (no value), rcl:R0603
- added SOLAR: M02PTH, SparkFun-Connectors:1X02
- C2: device rcl:E5-5 -> rcl:C0603
- moved U$4 23.1 mm to (1.65, 16.8), flipped to the bottom
- moved JP1 21.8 mm to (23.1, 22.1)
- moved J1 21.5 mm to (18.0, 21.3), turned to 180 degrees
- moved DF 18.2 mm to (3.56, 6.35), turned to 180 degrees
- moved J2 16.5 mm to (3.30, 20.3)
- moved U$1 16.0 mm to (15.2, 4.57), turned to 270 degrees
- moved U$2 14.7 mm to (4.32, 11.9), turned to 270 degrees
- moved U$3 11.9 mm to (8.64, 4.57), turned to 180 degrees
- moved R1 10.8 mm to (7.11, 9.40), turned to 90 degrees
- moved C2 10.7 mm to (4.32, 14.7), turned to 180 degrees
- moved R2 5.38 mm to (8.89, 9.40), turned to 270 degrees
- moved C1 3.31 mm to (14.5, 11.2)
Connections:
- new net N$5: D1.A, SOLAR.1
- net GND: now also C2.2, SOLAR.2; no longer C2.-
- net N$4: now also R3.1
- net VBATT: now also C2.1, D1.C, R3.2; no longer C2.+
Routing:
- net VCC: track 0.00 -> 46.3 mm, vias 0 -> 1
- net RESET: track 0.00 -> 44.3 mm, vias 0 -> 2
- net MOSI: track 0.00 -> 42.0 mm, vias 0 -> 1
- net DET/SCK: track 0.00 -> 32.9 mm, vias 0 -> 1
- net MISO: track 0.00 -> 31.4 mm, vias 0 -> 1
- net VBATT: track 0.00 -> 22.2 mm
- net N$4: track 0.00 -> 21.9 mm
- net RFM_SS: track 0.00 -> 11.7 mm, vias 0 -> 1
- net N$3: track 0.00 -> 10.0 mm
- net N$1: track 0.00 -> 8.01 mm
- net N$2: track 0.00 -> 5.00 mm
- net N$5: track 0.00 -> 3.12 mm
- added copper zone on layer 1, net GND
- added copper zone on layer 16, net GND
Other:
- board size 25 x 25 mm -> 50 x 24 mm
- board text added: "UKHASNET"
