File: pcb/node.sch (EAGLE design)
At the start: 10 parts, among them J1 AVR_SPI_PRG_62X3_LOCK

Commit message: placing parts
Parts:
- added C1: 100u, rcl:CPOL-EUSANYO_SMD_C6
- added C2: 4u7, rcl:CPOL-EUE5-5
Connections:
- net GND: now also C1.-, C2.-
- net VBATT: now also C2.+
- net VCC: now also C1.+
Changed lines of the file:
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@@
 <setting verticaltext="up"/>
 </settings>
-<grid distance="0.1" unitdist="inch" unit="inch" style="lines" multiple="1" display="yes" altdistance="0.005" altunitdist="inch" altunit="inch"/>
+<grid distance="0.1" unitdist="inch" unit="inch" style="lines" multiple="1" display="no" altdistance="0.01" altunitdist="inch" altunit="inch"/>
 <layers>
 <layer number="1" name="Top" color="4" fill="1" visible="no" active="no"/>
@@
 <part name="GND6" library="SparkFun-Aesthetics" deviceset="GND" device=""/>
 <part name="JP1" library="SparkFun-Connectors" deviceset="M01" device="PTH"/>
+<part name="C1" library="rcl" deviceset="CPOL-EU" device="SANYO_SMD_C6" value="100u"/>
+<part name="C2" library="rcl" deviceset="CPOL-EU" device="E5-5" value="4u7"/>
 </parts>
 <sheets>
@@
 <instance part="GND6" gate="1" x="198.12" y="12.7"/>
 <instance part="JP1" gate="G$1" x="208.28" y="22.86" rot="R180"/>
+<instance part="C1" gate="G$1" x="134.62" y="40.64"/>
+<instance part="C2" gate="G$1" x="83.82" y="33.02"/>
 </instances>
 <busses>
@@
 <wire x1="127" y1="27.94" x2="101.6" y2="27.94" width="0.1524" layer="91"/>
 <junction x="101.6" y="27.94"/>
+<pinref part="C1" gate="G$1" pin="-"/>
+<wire x1="134.62" y1="35.56" x2="134.62" y2="27.94" width="0.1524" layer="91"/>
+<wire x1="134.62" y1="27.94" x2="127" y2="27.94" width="0.1524" layer="91"/>
+<junction x="127" y="27.94"/>
+<pinref part="C2" gate="G$1" pin="-"/>
+<wire x1="83.82" y1="27.94" x2="101.6" y2="27.94" width="0.1524" layer="91"/>
 </segment>
 <segment>
@@
 <pinref part="R1" gate="G$1" pin="2"/>
 <junction x="127" y="48.26"/>
+<pinref part="C1" gate="G$1" pin="+"/>
+<wire x1="127" y1="48.26" x2="134.62" y2="48.26" width="0.1524" layer="91"/>
+<wire x1="134.62" y1="48.26" x2="134.62" y2="43.18" width="0.1524" layer="91"/>
 </segment>
 <segment>
@@
 <wire x1="83.82" y1="48.26" x2="86.36" y2="48.26" width="0.1524" layer="91"/>
 <label x="83.82" y="55.88" size="1.27" layer="95" rot="R180" xref="yes"/>
-</segment>
-</net>
+<wire x1="83.82" y1="48.26" x2="83.82" y2="35.56" width="0.1524" layer="91"/>
+<junction x="83.82" y="48.26"/>
+<pinref part="C2" gate="G$1" pin="+"/>
+</segment>
+</net>

Commit message: routing commence
Parts:
- added D1: (no value), dtb:DIODE-SOD123
- added R3: (no value), rcl:R-EU_R0603
- added SOLAR: M02PTH, SparkFun-Connectors:M02PTH
- C2: device rcl:CPOL-EUE5-5 -> rcl:C-EUC0603
Connections:
- new net N$5: D1.A, SOLAR.1
- net GND: now also C2.2, SOLAR.2; no longer C2.-
- net N$4: now also R3.1
- net VBATT: now also C2.1, D1.C, R3.2; no longer C2.+
Changed lines of the file:
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@@
 <?xml version="1.0" encoding="utf-8"?>
 <!DOCTYPE eagle SYSTEM "eagle.dtd">
-<eagle version="6.6.0">
+<eagle version="6.5.0">
 <drawing>
 <settings>
@@
 <layer number="20" name="Dimension" color="15" fill="1" visible="no" active="no"/>
 <layer number="21" name="tPlace" color="16" fill="1" visible="no" active="no"/>
-<layer number="22" name="bPlace" color="7" fill="1" visible="no" active="no"/>
+<layer number="22" name="bPlace" color="14" fill="1" visible="no" active="no"/>
 <layer number="23" name="tOrigins" color="15" fill="1" visible="no" active="no"/>
 <layer number="24" name="bOrigins" color="15" fill="1" visible="no" active="no"/>
@@
 <layer number="49" name="Reference" color="7" fill="1" visible="no" active="no"/>
 <layer number="50" name="dxf" color="7" fill="1" visible="no" active="no"/>
-<layer number="51" name="tDocu" color="14" fill="1" visible="no" active="no"/>
+<layer number="51" name="tDocu" color="6" fill="1" visible="no" active="no"/>
 <layer number="52" name="bDocu" color="7" fill="1" visible="no" active="no"/>
 <layer number="53" name="tGND_GNDA" color="7" fill="9" visible="no" active="no"/>
@@
 <part name="GND6" library="SparkFun-Aesthetics" deviceset="GND" device=""/>
 <part name="JP1" library="SparkFun-Connectors" deviceset="M01" device="PTH"/>
+<part name="C2" library="rcl" deviceset="C-EU" device="C0603" value="4u7"/>
+<part name="SOLAR" library="SparkFun-Connectors" deviceset="M02" device="PTH"/>
+<part name="D1" library="dtb" deviceset="DIODE-" device="SOD123"/>
+<part name="GND7" library="SparkFun-Aesthetics" deviceset="GND" device=""/>
 <part name="C1" library="rcl" deviceset="CPOL-EU" device="SANYO_SMD_C6" value="100u"/>
-<part name="C2" library="rcl" deviceset="CPOL-EU" device="E5-5" value="4u7"/>
+<part name="R3" library="rcl" deviceset="R-EU_" device="R0603"/>
 </parts>
 <sheets>
@@
 <instance part="GND6" gate="1" x="198.12" y="12.7"/>
 <instance part="JP1" gate="G$1" x="208.28" y="22.86" rot="R180"/>
+<instance part="C2" gate="G$1" x="83.82" y="33.02"/>
+<instance part="SOLAR" gate="G$1" x="-25.4" y="10.16"/>
+<instance part="D1" gate="G$1" x="-5.08" y="10.16"/>
+<instance part="GND7" gate="1" x="-12.7" y="12.7" rot="R90"/>
 <instance part="C1" gate="G$1" x="134.62" y="40.64"/>
-<instance part="C2" gate="G$1" x="83.82" y="33.02"/>
+<instance part="R3" gate="G$1" x="73.66" y="45.72" rot="R90"/>
 </instances>
 <busses>
@@
 <wire x1="127" y1="27.94" x2="101.6" y2="27.94" width="0.1524" layer="91"/>
 <junction x="101.6" y="27.94"/>
-<pinref part="C1" gate="G$1" pin="-"/>
 <wire x1="134.62" y1="35.56" x2="134.62" y2="27.94" width="0.1524" layer="91"/>
 <wire x1="134.62" y1="27.94" x2="127" y2="27.94" width="0.1524" layer="91"/>
 <junction x="127" y="27.94"/>
-<pinref part="C2" gate="G$1" pin="-"/>
+<pinref part="C2" gate="G$1" pin="2"/>
 <wire x1="83.82" y1="27.94" x2="101.6" y2="27.94" width="0.1524" layer="91"/>
+<pinref part="C1" gate="G$1" pin="-"/>
 </segment>
 <segment>
@@
 <junction x="198.12" y="17.78"/>
 </segment>
+<segment>
+<pinref part="GND7" gate="1" pin="GND"/>
+<pinref part="SOLAR" gate="G$1" pin="2"/>
+<wire x1="-15.24" y1="12.7" x2="-17.78" y2="12.7" width="0.1524" layer="91"/>
+</segment>
 </net>
 <net name="VCC" class="0">
@@
 <pinref part="R1" gate="G$1" pin="2"/>
 <junction x="127" y="48.26"/>
-<pinref part="C1" gate="G$1" pin="+"/>
 <wire x1="127" y1="48.26" x2="134.62" y2="48.26" width="0.1524" layer="91"/>
 <wire x1="134.62" y1="48.26" x2="134.62" y2="43.18" width="0.1524" layer="91"/>
+<pinref part="C1" gate="G$1" pin="+"/>
 </segment>
 <segment>
@@
 <segment>
 <pinref part="U$1" gate="G$1" pin="PB3(ADC3)"/>
-<wire x1="55.88" y1="40.64" x2="81.28" y2="40.64" width="0.1524" layer="91"/>
+<wire x1="55.88" y1="40.64" x2="73.66" y2="40.64" width="0.1524" layer="91"/>
+<wire x1="73.66" y1="40.64" x2="81.28" y2="40.64" width="0.1524" layer="91"/>
 <wire x1="81.28" y1="40.64" x2="81.28" y2="43.18" width="0.1524" layer="91"/>
 <pinref part="U$2" gate="G$1" pin="EN"/>
 <wire x1="81.28" y1="43.18" x2="86.36" y2="43.18" width="0.1524" layer="91"/>
+<pinref part="R3" gate="G$1" pin="1"/>
+<junction x="73.66" y="40.64"/>
 </segment>
 </net>
@@
 <pinref part="DF" gate="G$1" pin="P$1"/>
 <wire x1="86.36" y1="60.96" x2="83.82" y2="60.96" width="0.1524" layer="91"/>
-<wire x1="83.82" y1="60.96" x2="83.82" y2="48.26" width="0.1524" layer="91"/>
+<wire x1="83.82" y1="60.96" x2="83.82" y2="53.34" width="0.1524" layer="91"/>
 <pinref part="U$2" gate="G$1" pin="VIN"/>
+<wire x1="83.82" y1="53.34" x2="83.82" y2="48.26" width="0.1524" layer="91"/>
 <wire x1="83.82" y1="48.26" x2="86.36" y2="48.26" width="0.1524" layer="91"/>
 <label x="83.82" y="55.88" size="1.27" layer="95" rot="R180" xref="yes"/>
 <wire x1="83.82" y1="48.26" x2="83.82" y2="35.56" width="0.1524" layer="91"/>
 <junction x="83.82" y="48.26"/>
-<pinref part="C2" gate="G$1" pin="+"/>
+<pinref part="C2" gate="G$1" pin="1"/>
+<pinref part="R3" gate="G$1" pin="2"/>
+<wire x1="73.66" y1="50.8" x2="73.66" y2="53.34" width="0.1524" layer="91"/>
+<wire x1="73.66" y1="53.34" x2="83.82" y2="53.34" width="0.1524" layer="91"/>
+<junction x="83.82" y="53.34"/>
+</segment>
+<segment>
+<pinref part="D1" gate="G$1" pin="C"/>
+<wire x1="-2.54" y1="10.16" x2="5.08" y2="10.16" width="0.1524" layer="91"/>
+<label x="5.08" y="10.16" size="1.27" layer="95" xref="yes"/>
 </segment>
 </net>
@@
 </segment>
 </net>
+<net name="N$5" class="0">
+<segment>
+<pinref part="SOLAR" gate="G$1" pin="1"/>
+<pinref part="D1" gate="G$1" pin="A"/>
+<wire x1="-17.78" y1="10.16" x2="-7.62" y2="10.16" width="0.1524" layer="91"/>
+</segment>
+</net>
