File: fc-node/pcb/node.brd (EAGLE design)
At the start: 50 x 24 mm, 20 parts, among them IC1 HTU21D, J1 AVR_SPI_PRG_62X3_LOCK

Commit message: put things in the right places
Parts:
- removed C3: 100n, rcl:C0603
- removed IC1: HTU21D, Mine:DFN6-L
- removed R4, R5, R6: (no value), rcl:R0603
- U$1: value ATTINY84 -> ATTINY13SOIC; device SparkFun-DigitalIC:SO14 -> SparkFun-DigitalIC:SO08
- moved U$3 4.34 mm to (8.64, 4.57)
- moved R2 3.64 mm to (8.89, 9.65)
- moved R1 3.54 mm to (7.37, 9.65)
- moved C1 2.90 mm to (14.5, 11.2), turned to 0 degrees
- moved U$1 1.30 mm to (15.2, 4.57), turned to 270 degrees
- moved R3 1.27 mm to (4.06, 2.54)
- moved J2 1.14 mm to (3.30, 20.3), turned to 270 degrees
- moved D1 1.05 mm to (8.64, 16.3)
- moved DF 1.02 mm to (3.56, 6.35)
- moved JP1 1.02 mm to (23.1, 22.1)
- moved J1 0.76 mm to (18.0, 21.3)
- moved SOLAR 0.25 mm to (9.14, 18.8)
Connections:
- removed net DET: U$1.5, U$3.1
- removed net DIO0: U$1.12, U$4.DIO0
- removed net EN: R3.1, U$1.10, U$2.3
- removed net N$6: U$1.6
- removed net N$7: U$4.RESET
- removed net SCK: IC1.6, J1.3, U$1.9, U$4.SCK
- removed net VSENSE: R5.1, R6.2, U$1.13
- new net DET/SCK: J1.3, U$1.7, U$3.1, U$4.SCK
- net GND: now also U$1.4; no longer C3.2, IC1.2, R6.1, U$1.14
- net MISO: now also U$1.6; no longer U$1.8
- net MOSI: now also U$1.5; no longer IC1.1, U$1.7
- net N$4: now also R3.1, U$1.2, U$2.3; no longer U$1.3
- net RESET: now also U$1.1; no longer U$1.4
- net RFM_SS: now also U$1.3; no longer R4.1, U$1.11
- net VBATT: no longer R5.2
- net VCC: now also U$1.8; no longer C3.1, IC1.5, R4.2, U$1.1
Routing:
- net SCK: track 49.6 -> 0.00 mm, vias 2 -> 0
- net EN: track 35.6 -> 0.00 mm
- net DET/SCK: track 0.00 -> 32.9 mm, vias 0 -> 1
- net N$4: track 0.00 -> 21.9 mm
- net DIO0: track 20.7 -> 0.00 mm, vias 1 -> 0
- net RESET: track 25.6 -> 44.3 mm, vias 0 -> 2
- net VCC: track 61.9 -> 45.5 mm, vias 0 -> 1
- net DET: track 16.0 -> 0.00 mm
- net VBATT: track 35.2 -> 22.2 mm
- net MISO: track 21.1 -> 31.4 mm
- net MOSI: track 49.9 -> 42.0 mm, vias 2 -> 1
- net GND: track 5.75 -> 2.09 mm, vias 32 -> 21
- net RFM_SS: track 9.28 -> 11.7 mm
- net N$3: track 8.58 -> 10.0 mm
- net N$1: track 6.92 -> 8.26 mm
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Other:
- outline, holes or cut-outs redrawn
- board text added: "MAR '15"
- board text added: "UKHASNET"
- board text removed: "APR 15"
- board text removed: "APRIL 2015"
- board text removed: "JON"
- board text removed: "JON SOWMAN"
- board text removed: "SOWMAN"
- board text removed: "UKHAS"
- board text removed: "ukhas.net"
