File: fc-node/pcb/node.sch (EAGLE design)
At the start: 20 parts, among them IC1 HTU21D, J1 AVR_SPI_PRG_62X3_LOCK

Commit message: put things in the right places
Parts:
- removed C3: 100n, rcl:C-EUC0603
- removed IC1: HTU21D, Mine:HTU21D
- removed R4, R5, R6: (no value), rcl:R-EU_R0603
- U$1: value ATTINY84 -> ATTINY13SOIC; device SparkFun-DigitalIC:ATTINY84 -> SparkFun-DigitalIC:ATTINY13SOIC
Connections:
- removed net DET: U$1.(PCINT10/INT0/OC0A/CKOUT)PB2, U$3.DETECT
- removed net DIO0: U$1.(PCINT1/AIN0/ADC1)PA1, U$4.DIO0
- removed net EN: R3.1, U$1.(PCINT3/T0/ADC3)PA3, U$2.EN
- removed net N$6: U$1.(PCINT7/ICP/OC0B/ADC7)PA7
- removed net N$7: U$4.RESET
- removed net SCK: IC1.SCK, J1.3, U$1.(PCINT4/T1/SCL/USCK/ADC4)PA4, U$4.SCK
- removed net VSENSE: R5.1, R6.2, U$1.(PCINT0/AREF/ADC0)PA0
- new net DET/SCK: J1.3, U$1.PB2(SCK/ADC1), U$3.DETECT, U$4.SCK
- net GND: no longer C3.2, IC1.GND, R6.1
- net MISO: now also U$1.PB1(MISO); no longer U$1.(PCINT5/OC1B/MISO/DO/ADC5)PA5
- net MOSI: now also U$1.PB0(MOSI); no longer IC1.DATA, U$1.(PCINT6/OC1A/SDA/MOSI/ADC6)PA6
- net N$4: now also R3.1, U$1.PB3(ADC3), U$2.EN; no longer U$1.(PCINT9/XTAL2)PB1
- net RESET: now also U$1.PB5(NRES); no longer U$1.(PCINT11/~RESET/DW)PB3
- net RFM_SS: now also U$1.PB4(ADC2); no longer R4.1, U$1.(PCINT2/AIN1/ADC2)PA2
- net VBATT: no longer R5.2
- net VCC: no longer C3.1, IC1.VDD, R4.2
