File: pnode/pnode.brd (EAGLE design)
At the start: 50 x 23 mm, 39 parts, among them IC2 HTU21D, IC3 SI4012

Commit message: routing pnode
Parts:
- moved C2 12.1 mm to (20.6, 2.54), turned to 270 degrees
- moved R2 5.99 mm to (29.0, 13.5), turned to 90 degrees
- moved C13 5.68 mm to (35.8, 7.62), turned to 270 degrees
- moved C1 5.52 mm to (36.6, 13.5), turned to 90 degrees
- moved R8 3.38 mm to (30.2, 7.62), turned to 90 degrees
- moved R3 3.33 mm to (31.5, 13.5), turned to 270 degrees
- moved R6 3.05 mm to (34.0, 13.5), turned to 90 degrees
- moved R7 2.99 mm to (33.0, 7.62), turned to 270 degrees
- moved R5 1.91 mm to (17.3, 6.86)
- moved R4 1.91 mm to (15.2, 6.86)
- moved C4 1.90 mm to (13.2, 6.86), turned to 90 degrees
- moved C3 1.42 mm to (22.6, 2.54)
- moved C8 1.35 mm to (17.3, 11.2)
- moved L1 1.35 mm to (15.2, 11.2)
- moved C7 1.34 mm to (13.2, 11.2), turned to 90 degrees
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Routing:
- net +3V3: track 0.00 -> 87.8 mm, vias 0 -> 2
- net NRST: track 0.00 -> 27.1 mm, vias 0 -> 2
- net SDA: track 0.00 -> 26.3 mm
- net SWCLK: track 0.00 -> 21.1 mm, vias 0 -> 2
- net SCL: track 0.00 -> 21.0 mm, vias 0 -> 2
- net VBATT: track 0.00 -> 20.9 mm
- net N$2: track 0.00 -> 20.6 mm
- net SWDAT: track 0.00 -> 17.7 mm, vias 0 -> 2
- net CLAMP: track 0.00 -> 17.2 mm
- net GND: track 0.00 -> 16.7 mm, vias 0 -> 50
- net VBATT_MEAS: track 0.00 -> 15.0 mm
- net N$4: track 0.00 -> 13.7 mm
- net RADIO_SHDN: track 0.00 -> 10.3 mm, vias 0 -> 2
- net N$1: track 0.00 -> 9.34 mm
- net N$5: track 0.00 -> 7.73 mm
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- added copper zone on layer 1, net GND
- added copper zone on layer 16, net GND

Commit message: Routing and tidying + silk
Parts:
- moved C13 1.02 mm to (34.8, 7.62)
- moved R7 0.51 mm to (32.5, 7.62)
- moved L4 0.51 mm to (9.12, 16.0)
- moved L2 0.12 mm to (11.4, 15.0), turned to 270 degrees
- moved L5 0.11 mm to (11.4, 17.0), turned to 90 degrees
Routing:
- net VBATT_MEAS: track 15.0 -> 14.0 mm
- net GND: track 16.7 -> 17.7 mm, vias 50 -> 53
- net N$4: track 13.7 -> 12.8 mm, vias 0 -> 2
- net N$8: track 6.27 -> 5.51 mm
- net N$7: track 4.95 -> 4.44 mm
Other:
- board text added: "JON"
- board text added: "M0JSN"
- board text added: "SOWMAN"
- board text added: "UKHASnet"
- board text added: "ukhas.net"

Commit message: Tidying up silk
Parts:
- moved H1 0.35 mm to (46.0, 19.0)
- moved H2 0.35 mm to (46.0, 4.00)
- moved H3 0.35 mm to (4.00, 4.00)
- moved H4 0.35 mm to (4.00, 19.0)
- moved C13 0.25 mm to (34.5, 7.62)
- moved U$1 0.25 mm to (44.7, 11.2)
- moved R7 0.25 mm to (32.3, 7.62)
- moved R8 0.25 mm to (30.0, 7.62)
Other:
- board text added: "Jan 2016"
Changed lines of the file:
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@@
 <wire x1="50" y1="2" x2="50" y2="21" width="0" layer="20"/>
 <wire x1="50" y1="21" x2="48" y2="23" width="0" layer="20" curve="90"/>
-<dimension x1="0" y1="23" x2="0" y2="0" x3="-10.25" y3="11.5" textsize="1.778" layer="51"/>
-<dimension x1="0" y1="23" x2="50" y2="23" x3="25" y3="32" textsize="1.778" layer="51"/>
 <text x="9.144" y="0.508" size="1.27" layer="21" font="vector" ratio="15" rot="R90">UKHASnet</text>
 <text x="11.176" y="2.032" size="1.27" layer="21" font="vector" ratio="15" rot="R90">M0JSN</text>
-<text x="36.576" y="8.382" size="1.27" layer="21" font="vector" ratio="15">JON</text>
-<text x="36.576" y="6.604" size="1.27" layer="21" font="vector" ratio="15">SOWMAN</text>
-<text x="19.812" y="16.51" size="1.27" layer="21" font="vector" ratio="15">ukhas.net</text>
+<text x="21.082" y="16.51" size="1.27" layer="21" font="vector" ratio="15">JON</text>
+<text x="19.558" y="14.732" size="1.27" layer="21" font="vector" ratio="15">SOWMAN</text>
+<text x="18.542" y="13.208" size="1.27" layer="21" font="vector" ratio="15">Jan 2016</text>
+<text x="35.56" y="7.366" size="1.27" layer="21" font="vector" ratio="15">ukhas.net</text>
 </plain>
 <attributes>
@@
 </element>
 <element name="U$3" library="jonsowman" package="SWD_PTH_SHROUD" value="SWD_PTH_SHROUD" x="33.02" y="20.32"/>
-<element name="U$1" library="jonsowman" package="13MM_DC_JACK" value="13MM_DC_JACKPTH" x="44.704" y="11.43" smashed="yes" rot="R180"/>
+<element name="U$1" library="jonsowman" package="13MM_DC_JACK" value="13MM_DC_JACKPTH" x="44.704" y="11.176" smashed="yes" rot="R180"/>
 <element name="R1" library="passives-7351" package="R0603-N" value="100R" x="39.116" y="13.462" smashed="yes" rot="R270">
 <attribute name="NAME" x="39.91290625" y="15.864921875" size="0.8128" layer="25" font="vector" ratio="13" rot="R180"/>
@@
 <attribute name="NAME" x="37.37290625" y="15.864921875" size="0.8128" layer="25" font="vector" ratio="13" rot="R180"/>
 </element>
-<element name="R7" library="passives-7351" package="R0603-N" value="1M" x="32.512" y="7.62" smashed="yes" rot="R270">
-<attribute name="NAME" x="33.30890625" y="10.022921875" size="0.8128" layer="25" font="vector" ratio="13" rot="R180"/>
-</element>
-<element name="R8" library="passives-7351" package="R0603-N" value="1M" x="30.226" y="7.62" smashed="yes" rot="R90">
-<attribute name="NAME" x="31.02290625" y="10.022921875" size="0.8128" layer="25" font="vector" ratio="13" rot="R180"/>
+<element name="R7" library="passives-7351" package="R0603-N" value="1M" x="32.258" y="7.62" smashed="yes" rot="R270">
+<attribute name="NAME" x="33.05490625" y="10.022921875" size="0.8128" layer="25" font="vector" ratio="13" rot="R180"/>
+</element>
+<element name="R8" library="passives-7351" package="R0603-N" value="1M" x="29.972" y="7.62" smashed="yes" rot="R90">
+<attribute name="NAME" x="30.76890625" y="10.022921875" size="0.8128" layer="25" font="vector" ratio="13" rot="R180"/>
 </element>
 <element name="C2" library="passives-7351" package="C0603-N" value="100n" x="20.574" y="2.54" smashed="yes" rot="R270">
@@
 </element>
 <element name="J$1" library="jonsowman" package="SMA-EDGE" value="SMA_EDGE" x="2.286" y="8.89" rot="R90"/>
-<element name="H1" library="dtb" package="3,0-PAD" value="MOUNT-PAD-ROUND3.0" x="46.25" y="19.25"/>
-<element name="H2" library="dtb" package="3,0-PAD" value="MOUNT-PAD-ROUND3.0" x="46.25" y="3.75"/>
-<element name="H3" library="dtb" package="3,0-PAD" value="MOUNT-PAD-ROUND3.0" x="3.75" y="3.75"/>
-<element name="H4" library="dtb" package="3,0-PAD" value="MOUNT-PAD-ROUND3.0" x="3.75" y="19.25"/>
+<element name="H1" library="dtb" package="3,0-PAD" value="MOUNT-PAD-ROUND3.0" x="46" y="19"/>
+<element name="H2" library="dtb" package="3,0-PAD" value="MOUNT-PAD-ROUND3.0" x="46" y="4"/>
+<element name="H3" library="dtb" package="3,0-PAD" value="MOUNT-PAD-ROUND3.0" x="4" y="4"/>
+<element name="H4" library="dtb" package="3,0-PAD" value="MOUNT-PAD-ROUND3.0" x="4" y="19"/>
 <element name="C3" library="passives-7351" package="C0603-N" value="1u" x="22.606" y="2.54" smashed="yes" rot="R90">
 <attribute name="NAME" x="23.40290625" y="4.942921875" size="0.8128" layer="25" font="vector" ratio="13" rot="R180"/>
@@
 <attribute name="NAME" x="27.46690625" y="4.942921875" size="0.8128" layer="25" font="vector" ratio="13" rot="R180"/>
 </element>
-<element name="C13" library="passives-7351" package="C0603-N" value="1u" x="34.798" y="7.62" smashed="yes" rot="R270">
-<attribute name="NAME" x="36.10290625" y="10.022921875" size="0.8128" layer="25" font="vector" ratio="13" rot="R180"/>
+<element name="C13" library="passives-7351" package="C0603-N" value="1u" x="34.544" y="7.62" smashed="yes" rot="R270">
+<attribute name="NAME" x="35.84890625" y="10.022921875" size="0.8128" layer="25" font="vector" ratio="13" rot="R180"/>
 </element>
 </elements>
@@
 <wire x1="11.914" y1="20.942" x2="11.402" y2="20.942" width="0.4064" layer="1"/>
 <wire x1="11.402" y1="20.942" x2="9.878" y2="19.418" width="0.4064" layer="1"/>
-<wire x1="34.798" y1="6.82" x2="36.36" y2="6.82" width="0.4064" layer="1"/>
+<wire x1="34.544" y1="6.82" x2="36.36" y2="6.82" width="0.4064" layer="1"/>
 <wire x1="36.36" y1="6.82" x2="38.608" y2="4.572" width="0.4064" layer="1"/>
 <wire x1="38.608" y1="4.572" x2="38.608" y2="3.318" width="0.4064" layer="1"/>
@@
 <via x="28.448" y="3.048" extent="1-16" drill="0.381"/>
 <via x="28.194" y="9.398" extent="1-16" drill="0.381"/>
-<via x="37.846" y="11.684" extent="1-16" drill="0.381"/>
+<via x="37.846" y="11.938" extent="1-16" drill="0.381"/>
 <via x="35.306" y="11.684" extent="1-16" drill="0.381"/>
 <via x="27.432" y="16.256" extent="1-16" drill="0.381"/>
@@
 <via x="14.224" y="18.288" extent="1-16" drill="0.381"/>
 <via x="12.954" y="22.098" extent="1-16" drill="0.381"/>
-<via x="39.624" y="10.922" extent="1-16" drill="0.381"/>
-<via x="41.656" y="8.636" extent="1-16" drill="0.381"/>
-<via x="40.386" y="15.24" extent="1-16" drill="0.381"/>
-<via x="42.672" y="15.24" extent="1-16" drill="0.381"/>
-<via x="40.386" y="13.462" extent="1-16" drill="0.381"/>
+<via x="39.497" y="11.049" extent="1-16" drill="0.381"/>
+<via x="41.402" y="8.636" extent="1-16" drill="0.381"/>
+<via x="40.386" y="15.113" extent="1-16" drill="0.381"/>
+<via x="42.672" y="15.113" extent="1-16" drill="0.381"/>
+<via x="40.386" y="13.208" extent="1-16" drill="0.381"/>
 <via x="35.306" y="14.478" extent="1-16" drill="0.381"/>
 <via x="21.336" y="7.62" extent="1-16" drill="0.381"/>
@@
 <contactref element="L1" pad="1"/>
 <contactref element="L5" pad="2"/>
-<wire x1="15.24" y1="11.976" x2="17.272" y2="11.976" width="0.254" layer="1"/>
+<wire x1="15.24" y1="11.976" x2="17.272" y2="11.976" width="0.4064" layer="1"/>
 <wire x1="15.24" y1="11.976" x2="14.948" y2="11.976" width="0.4064" layer="1"/>
 <wire x1="14.948" y1="11.976" x2="13.589" y2="13.335" width="0.4064" layer="1"/>
@@
 <wire x1="32.512" y1="1.016" x2="32.512" y2="2.37" width="0.4064" layer="1"/>
 <wire x1="32.512" y1="2.37" x2="32.342" y2="2.54" width="0.4064" layer="1"/>
-<wire x1="32.512" y1="6.82" x2="32.512" y2="2.71" width="0.4064" layer="1"/>
 <wire x1="32.512" y1="2.71" x2="32.342" y2="2.54" width="0.4064" layer="1"/>
+<wire x1="32.258" y1="6.82" x2="32.342" y2="6.82" width="0.4064" layer="1"/>
+<wire x1="32.342" y1="6.82" x2="32.342" y2="2.54" width="0.4064" layer="1"/>
 </signal>
 <signal name="SWDAT">
@@
 <contactref element="R1" pad="2"/>
 <contactref element="R6" pad="2"/>
-<wire x1="41.734" y1="11.9" x2="42.204" y2="11.43" width="0.4064" layer="1"/>
-<wire x1="41.734" y1="11.9" x2="39.878" y2="11.9" width="0.3048" layer="1"/>
+<wire x1="41.48" y1="11.9" x2="42.204" y2="11.176" width="0.4064" layer="1"/>
+<wire x1="41.48" y1="11.9" x2="39.878" y2="11.9" width="0.3048" layer="1"/>
 <wire x1="39.878" y1="11.9" x2="39.116" y2="12.662" width="0.3048" layer="1"/>
 <wire x1="39.116" y1="12.662" x2="38.392" y2="12.662" width="0.3048" layer="1"/>
@@
 <contactref element="R2" pad="2"/>
 <contactref element="R3" pad="1"/>
-<wire x1="44.704" y1="14.23" x2="39.148" y2="14.23" width="0.3048" layer="1"/>
 <wire x1="39.148" y1="14.23" x2="39.116" y2="14.262" width="0.254" layer="1"/>
 <wire x1="28.956" y1="14.262" x2="31.496" y2="14.262" width="0.3048" layer="1"/>
@@
 <wire x1="33.02" y1="15.494" x2="37.884" y2="15.494" width="0.3048" layer="1"/>
 <wire x1="37.884" y1="15.494" x2="39.116" y2="14.262" width="0.3048" layer="1"/>
-<wire x1="47.204" y1="11.43" x2="47.204" y2="11.73" width="0.3048" layer="1"/>
-<wire x1="47.204" y1="11.73" x2="44.704" y2="14.23" width="0.3048" layer="1"/>
+<wire x1="47.204" y1="11.176" x2="47.204" y2="11.73" width="0.3048" layer="1"/>
+<wire x1="47.204" y1="11.73" x2="44.704" y2="13.976" width="0.3048" layer="1"/>
+<wire x1="39.148" y1="14.23" x2="44.45" y2="14.23" width="0.3048" layer="1"/>
+<wire x1="44.45" y1="14.23" x2="44.704" y2="13.976" width="0.3048" layer="1"/>
 </signal>
 <signal name="VBATT_MEAS">
@@
 <contactref element="R8" pad="2"/>
 <contactref element="C13" pad="1"/>
-<wire x1="34.798" y1="8.42" x2="32.512" y2="8.42" width="0.4064" layer="1"/>
-<wire x1="32.512" y1="8.42" x2="30.226" y2="8.42" width="0.4064" layer="1"/>
-<wire x1="30.226" y1="8.42" x2="28.232" y2="8.42" width="0.3048" layer="1"/>
+<wire x1="34.544" y1="8.42" x2="32.258" y2="8.42" width="0.4064" layer="1"/>
+<wire x1="32.258" y1="8.42" x2="29.972" y2="8.42" width="0.4064" layer="1"/>
+<wire x1="29.972" y1="8.42" x2="28.232" y2="8.42" width="0.3048" layer="1"/>
 <wire x1="28.232" y1="8.42" x2="27.178" y2="7.366" width="0.3048" layer="1"/>
 <wire x1="27.178" y1="7.366" x2="27.178" y2="5.08" width="0.3048" layer="1"/>

Commit message: Routing for pnodelv
Parts:
- moved U$3 0.25 mm to (33.0, 20.1)
Other:
- board text added: "3.5-6V"
- board text added: "SWD"
Changed lines of the file:
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@@
 <text x="18.542" y="13.208" size="1.27" layer="21" font="vector" ratio="15">Jan 2016</text>
 <text x="35.56" y="7.366" size="1.27" layer="21" font="vector" ratio="15">ukhas.net</text>
+<text x="37.846" y="18.542" size="1.27" layer="21" font="vector" ratio="15" rot="R90">SWD</text>
+<text x="42.164" y="0.508" size="1.27" layer="21" font="vector" ratio="15" rot="R90">3.5-6V</text>
 </plain>
 <attributes>
@@
 </class>
 </classes>
-<designrules name="dirt_cheap_dirty_boards.v1">
+<designrules name="dirt_cheap_dirty_boards.v1 *">
 <description language="en">&lt;b&gt;Dirty Cheap Dirty Board Design Rules&lt;/b&gt;
 &lt;br&gt;
@@
 <param name="dpGapFactor" value="2.5"/>
 <param name="checkGrid" value="0"/>
-<param name="checkAngle" value="0"/>
+<param name="checkAngle" value="1"/>
 <param name="checkFont" value="1"/>
 <param name="checkRestrict" value="0"/>
@@
 <attribute name="VALUE" x="28.067" y="4.445" size="1.27" layer="27" rot="R270"/>
 </element>
-<element name="U$3" library="jonsowman" package="SWD_PTH_SHROUD" value="SWD_PTH_SHROUD" x="33.02" y="20.32"/>
+<element name="U$3" library="jonsowman" package="SWD_PTH_SHROUD" value="SWD_PTH_SHROUD" x="33.02" y="20.066"/>
 <element name="U$1" library="jonsowman" package="13MM_DC_JACK" value="13MM_DC_JACKPTH" x="44.704" y="11.176" smashed="yes" rot="R180"/>
 <element name="R1" library="passives-7351" package="R0603-N" value="100R" x="39.116" y="13.462" smashed="yes" rot="R270">
@@
 <wire x1="23.297" y1="11.8078" x2="23.297" y2="9.398" width="0.4064" layer="1"/>
 <wire x1="23.297" y1="9.398" x2="23.297" y2="5.9722" width="0.3048" layer="1"/>
-<wire x1="30.48" y1="19.685" x2="30.099" y2="19.685" width="0.4064" layer="1"/>
-<wire x1="30.099" y1="19.685" x2="28.956" y2="20.828" width="0.4064" layer="1"/>
 <wire x1="28.956" y1="20.828" x2="27.178" y2="20.828" width="0.4064" layer="1"/>
 <wire x1="27.178" y1="20.828" x2="25.146" y2="18.796" width="0.4064" layer="1"/>
@@
 <wire x1="17.78" y1="13.208" x2="14.7149" y2="13.208" width="0.4064" layer="1"/>
 <wire x1="14.7149" y1="13.208" x2="13.0989" y2="14.824" width="0.4064" layer="1"/>
+<wire x1="30.48" y1="19.431" x2="30.353" y2="19.431" width="0.4064" layer="1"/>
+<wire x1="30.353" y1="19.431" x2="28.956" y2="20.828" width="0.4064" layer="1"/>
 </signal>
 <signal name="SCL">
@@
 <wire x1="12.319" y1="6.604" x2="12.319" y2="4.953" width="0.3048" layer="1"/>
 <wire x1="12.319" y1="4.953" x2="12.954" y2="4.318" width="0.3048" layer="1"/>
-<wire x1="12.954" y1="4.318" x2="13.216" y2="4.318" width="0.254" layer="1"/>
-<wire x1="13.216" y1="4.318" x2="13.486" y2="4.302" width="0.3048" layer="1"/>
 <wire x1="17.3251" y1="16.824" x2="16.57" y2="16.824" width="0.3048" layer="1"/>
 <wire x1="16.57" y1="16.824" x2="16.256" y2="16.51" width="0.3048" layer="1"/>
@@
 <wire x1="18.542" y1="14.732" x2="20.32" y2="14.732" width="0.3048" layer="1"/>
 <wire x1="20.32" y1="14.732" x2="20.828" y2="14.224" width="0.3048" layer="1"/>
+<wire x1="13.486" y1="4.302" x2="12.97" y2="4.302" width="0.3048" layer="1"/>
+<wire x1="12.97" y1="4.302" x2="12.954" y2="4.318" width="0.3048" layer="1"/>
 </signal>
 <signal name="N$4">
@@
 <wire x1="15.24" y1="11.976" x2="14.948" y2="11.976" width="0.4064" layer="1"/>
 <wire x1="14.948" y1="11.976" x2="13.589" y2="13.335" width="0.4064" layer="1"/>
-<wire x1="11.43" y1="17.498" x2="12.418" y2="17.498" width="0.4064" layer="1"/>
-<wire x1="12.418" y1="17.498" x2="12.319" y2="17.526" width="0.4064" layer="1"/>
 <via x="12.319" y="17.526" extent="1-16" drill="0.381"/>
 <wire x1="12.319" y1="17.526" x2="12.319" y2="14.224" width="0.4064" layer="16"/>
@@
 <wire x1="11.811" y1="13.335" x2="11.43" y2="13.716" width="0.4064" layer="1"/>
 <wire x1="11.43" y1="13.716" x2="11.43" y2="14.506" width="0.4064" layer="1"/>
+<wire x1="11.43" y1="17.498" x2="12.291" y2="17.498" width="0.4064" layer="1"/>
+<wire x1="12.291" y1="17.498" x2="12.319" y2="17.526" width="0.4064" layer="1"/>
 </signal>
 <signal name="N$7">
@@
 <wire x1="33.02" y1="2.71" x2="36" y2="2.71" width="0.4064" layer="1"/>
 <wire x1="36" y1="2.71" x2="36.592" y2="3.302" width="0.4064" layer="1"/>
-<wire x1="22.606" y1="1.74" x2="22.86" y2="1.524" width="0.4064" layer="1"/>
-<wire x1="22.86" y1="1.524" x2="23.876" y2="0.508" width="0.4064" layer="1"/>
 <wire x1="23.876" y1="0.508" x2="32.004" y2="0.508" width="0.4064" layer="1"/>
 <wire x1="32.004" y1="0.508" x2="32.512" y2="1.016" width="0.4064" layer="1"/>
@@
 <wire x1="32.258" y1="6.82" x2="32.342" y2="6.82" width="0.4064" layer="1"/>
 <wire x1="32.342" y1="6.82" x2="32.342" y2="2.54" width="0.4064" layer="1"/>
+<wire x1="22.606" y1="1.74" x2="22.644" y2="1.74" width="0.4064" layer="1"/>
+<wire x1="22.644" y1="1.74" x2="23.876" y2="0.508" width="0.4064" layer="1"/>
 </signal>
 <signal name="SWDAT">
@@
 <wire x1="24.638" y1="16.51" x2="24.638" y2="19.05" width="0.3048" layer="1"/>
 <wire x1="24.638" y1="19.05" x2="26.924" y2="21.336" width="0.3048" layer="1"/>
-<wire x1="26.924" y1="21.336" x2="30.099" y2="21.336" width="0.3048" layer="1"/>
-<wire x1="30.099" y1="21.336" x2="30.48" y2="20.955" width="0.3048" layer="1"/>
+<wire x1="26.924" y1="21.336" x2="29.845" y2="21.336" width="0.3048" layer="1"/>
+<wire x1="29.845" y1="21.336" x2="30.48" y2="20.701" width="0.3048" layer="1"/>
 </signal>
 <signal name="SWCLK">
@@
 <wire x1="26.67" y1="21.844" x2="31.242" y2="21.844" width="0.3048" layer="1"/>
 <wire x1="31.242" y1="21.844" x2="31.75" y2="21.336" width="0.3048" layer="1"/>
-<wire x1="31.75" y1="21.336" x2="31.75" y2="20.955" width="0.3048" layer="1"/>
+<wire x1="31.75" y1="21.336" x2="31.75" y2="20.701" width="0.3048" layer="1"/>
 <wire x1="19.558" y1="13.462" x2="19.812" y2="13.462" width="0.254" layer="16"/>
 <wire x1="19.812" y1="13.462" x2="20.32" y2="13.97" width="0.3048" layer="16"/>
@@
 <contactref element="U$3" pad="10"/>
 <contactref element="STM32" pad="4"/>
-<wire x1="35.56" y1="20.955" x2="35.941" y2="20.955" width="0.3048" layer="1"/>
-<wire x1="35.941" y1="20.955" x2="36.576" y2="20.32" width="0.3048" layer="1"/>
+<wire x1="35.56" y1="20.701" x2="36.195" y2="20.701" width="0.3048" layer="1"/>
+<wire x1="36.195" y1="20.701" x2="36.576" y2="20.32" width="0.3048" layer="1"/>
 <wire x1="36.576" y1="20.32" x2="36.576" y2="16.51" width="0.3048" layer="1"/>
 <wire x1="36.576" y1="16.51" x2="36.068" y2="16.002" width="0.3048" layer="1"/>
@@
 <wire x1="33.02" y1="15.494" x2="37.884" y2="15.494" width="0.3048" layer="1"/>
 <wire x1="37.884" y1="15.494" x2="39.116" y2="14.262" width="0.3048" layer="1"/>
-<wire x1="47.204" y1="11.176" x2="47.204" y2="11.73" width="0.3048" layer="1"/>
-<wire x1="47.204" y1="11.73" x2="44.704" y2="13.976" width="0.3048" layer="1"/>
 <wire x1="39.148" y1="14.23" x2="44.45" y2="14.23" width="0.3048" layer="1"/>
 <wire x1="44.45" y1="14.23" x2="44.704" y2="13.976" width="0.3048" layer="1"/>
+<wire x1="47.204" y1="11.176" x2="47.204" y2="11.476" width="0.3048" layer="1"/>
+<wire x1="47.204" y1="11.476" x2="44.704" y2="13.976" width="0.3048" layer="1"/>
 </signal>
 <signal name="VBATT_MEAS">
