File: fc-node2/pcb/node.sch (EAGLE design)
At the start: 15 parts, among them J1 AVR_SPI_PRG_62X3_LOCK

Commit message: put things in the right places
Parts:
- added C3: 100n, rcl:C-EUC0603
- added IC1: HTU21D, Mine:HTU21D
- added R4, R5, R6: (no value), rcl:R-EU_R0603
- U$1: value ATTINY13SOIC -> ATTINY84; device SparkFun-DigitalIC:ATTINY13SOIC -> SparkFun-DigitalIC:ATTINY84
Connections:
- removed net DET/SCK: J1.3, U$1.PB2(SCK/ADC1), U$3.DETECT, U$4.SCK
- new net DET: U$1.(PCINT10/INT0/OC0A/CKOUT)PB2, U$3.DETECT
- new net DIO0: U$1.(PCINT1/AIN0/ADC1)PA1, U$4.DIO0
- new net EN: R3.1, U$1.(PCINT3/T0/ADC3)PA3, U$2.EN
- new net N$6: U$1.(PCINT7/ICP/OC0B/ADC7)PA7
- new net N$7: U$4.RESET
- new net SCK: IC1.SCK, J1.3, U$1.(PCINT4/T1/SCL/USCK/ADC4)PA4, U$4.SCK
- new net VSENSE: R5.1, R6.2, U$1.(PCINT0/AREF/ADC0)PA0
- net GND: now also C3.2, IC1.GND, R6.1
- net MISO: now also U$1.(PCINT5/OC1B/MISO/DO/ADC5)PA5; no longer U$1.PB1(MISO)
- net MOSI: now also IC1.DATA, U$1.(PCINT6/OC1A/SDA/MOSI/ADC6)PA6; no longer U$1.PB0(MOSI)
- net N$4: now also U$1.(PCINT9/XTAL2)PB1; no longer R3.1, U$1.PB3(ADC3), U$2.EN
- net RESET: now also U$1.(PCINT11/~RESET/DW)PB3; no longer U$1.PB5(NRES)
- net RFM_SS: now also R4.1, U$1.(PCINT2/AIN1/ADC2)PA2; no longer U$1.PB4(ADC2)
- net VBATT: now also R5.2
- net VCC: now also C3.1, IC1.VDD, R4.2

Commit message: adapt fc2 to take 80mah nimh button cells with solder tabs
Parts:
- removed DF: 4u7, jonsowman:BOURNS_SRN5040
- removed J2: (no value), dtb:JST_2MM_MALE_TH
- removed U$3: BU49X_VDET_SOT235, jonsowman:BU49X_VDET_SOT235
- added JP2: (no value), SparkFun:M03PTH
- added L1: 4.7u, passives-7351:INDUCTOR0603-N
- C1: value 100u -> 4u7; device rcl:CPOL-EUSANYO_SMD_C6 -> rcl:C-EUC0603
- R5, R6: value (none) -> 4k7
Connections:
- removed net DET: U$1.(PCINT10/INT0/OC0A/CKOUT)PB2, U$3.DETECT
- removed net VSENSE: R5.1, R6.2, U$1.(PCINT0/AREF/ADC0)PA0
- net EN: no longer U$1.(PCINT3/T0/ADC3)PA3
- net GND: now also C1.2, JP2.1; no longer C1.-, J2.-, R6.1, U$3.GND
- net MOSI: now also R5.1
- net N$1: now also L1.P$2; no longer DF.P$2
- net SCK: now also R6.1
- net VBATT: now also JP2.3, L1.P$1, U$1.(PCINT0/AREF/ADC0)PA0; no longer DF.P$1, J2.+, R5.2
- net VCC: now also C1.1, R5.2, R6.2; no longer C1.+, U$3.VDD
Other:
- moved on the sheet: R5, R6
