File: rgb-node/pcb/node.brd (EAGLE design)
At the start: 54 x 17 mm, 19 parts, among them U2 MCP1640

Commit message: dumped some things on the pcb
Parts:
- moved D2 9.23 mm to (16.8, 4.32), turned to 90 degrees
- moved C2 6.59 mm to (48.3, 8.38), turned to 0 degrees
- moved TC1 4.58 mm to (11.4, 4.06), turned to 270 degrees
- moved C1 4.35 mm to (51.6, 11.9), turned to 0 degrees
- moved R2 4.34 mm to (48.3, 10.2), turned to 0 degrees
- moved R4 4.23 mm to (48.3, 6.60), turned to 180 degrees
- moved L1 3.34 mm to (51.6, 14.7), turned to 270 degrees
- moved U2 2.84 mm to (48.3, 14.7), turned to 90 degrees
- moved R1 2.29 mm to (48.3, 11.9), turned to 0 degrees
- moved BAT2 0.14 mm to (26.9, 8.50)

Commit message: dumped some things on the pcb 12
Parts:
- removed TP4, TP5, TP6, TP7: TEST-POINT3, SparkFun-Passives:PAD.03X.03
- moved L1 1.78 mm to (49.8, 14.7)
- moved R1 1.78 mm to (46.5, 11.9)
- moved U2 1.78 mm to (46.5, 14.7)
- moved C1 1.27 mm to (50.3, 11.9)
- turned C2 to 180 degrees
- turned R2 to 180 degrees
- turned R4 to 0 degrees
Connections:
- net MISO: now also U$1.12; no longer TP6.P$1
- net MOSI: now also U$1.13; no longer TP5.P$1
- net RFM_SS: now also U$1.10; no longer TP4.P$1
- net SCK: now also U$1.11; no longer TP7.P$1
Routing:
- net VCC: track 0.00 -> 60.5 mm, vias 0 -> 2
- net VBATT: track 0.00 -> 21.7 mm
- net N$3: track 0.00 -> 11.4 mm
- net N$2: track 0.00 -> 9.54 mm
- net GND: track 0.00 -> 2.48 mm
- net N$1: track 0.00 -> 2.21 mm

Commit message: commiting work on rgb-node
Parts:
- removed L1: 4.7u, passives-7351:L0603-N
- added C4: 10uF, SparkFun-Capacitors:CPOL-RADIAL-2.5MM-5MM
- added L2: 3.3µH/±20%/450mA, SparkFun-Coils:0805
- moved TC1 11.1 mm to (22.5, 4.06)
- moved TP1 11.0 mm to (14.4, 14.9)
- moved D2 7.70 mm to (9.14, 3.22), turned to 180 degrees
- moved JP1 6.86 mm to (58.9, 1.59)
- moved BAT2 5.08 mm to (32.0, 8.50)
- moved C1 5.00 mm to (55.3, 11.9)
- moved C2 5.00 mm to (53.3, 8.38)
- moved R1 5.00 mm to (51.5, 11.9)
- moved R2 5.00 mm to (53.3, 10.2)
- moved R4 5.00 mm to (53.3, 6.60)
- moved U$1 5.00 mm to (21.0, 13.0)
- moved U$4 5.00 mm to (26.6, 0.25)
- moved U2 5.00 mm to (51.5, 14.7)
- moved C3 5.00 mm to (16.2, 14.7)
Connections:
- new net VIB_SW: C4.1, U$1.6
- net GND: now also C4.2
- net N$1: now also L2.2; no longer L1.2
- net VBATT: now also L2.1; no longer L1.1
Routing:
- net VCC: track 60.5 -> 0.00 mm
- net VBATT: track 21.7 -> 0.00 mm
- net N$3: track 11.4 -> 0.00 mm
- net N$2: track 9.54 -> 0.00 mm
- net GND: track 2.48 -> 0.00 mm, vias 0 -> 2
- net N$1: track 2.21 -> 0.00 mm
Other:
- board size 54 x 17 mm -> 64 x 17 mm
- board text removed: "ICSP"
