File: rgb-node/pcb/node.sch (EAGLE design)
At the start: 19 parts, among them U2 MCP1640

Commit message: dumped some things on the pcb
Other:
- note removed: "Jon Sowman 04/17"
- note removed: "Low power film canister node with DS18B20"
Changed lines of the file:
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@@
 <setting verticaltext="up"/>
 </settings>
-<grid distance="0.05" unitdist="inch" unit="inch" style="lines" multiple="1" display="no" altdistance="0.01" altunitdist="inch" altunit="inch"/>
+<grid distance="0.1" unitdist="inch" unit="inch" style="lines" multiple="1" display="no" altdistance="0.01" altunitdist="inch" altunit="inch"/>
 <layers>
 <layer number="1" name="Top" color="4" fill="1" visible="no" active="no"/>
@@
 <part name="GND7" library="SparkFun-Aesthetics" deviceset="GND" device=""/>
 <part name="C3" library="passives-7351" deviceset="CAPACITOR" device="0603-N" value="100n"/>
+<part name="SUPPLY6" library="SparkFun-Aesthetics" deviceset="VCC" device=""/>
 </parts>
 <sheets>
 <sheet>
 <plain>
-<text x="124.46" y="-71.12" size="2.54" layer="94" font="vector" ratio="15">Low power film canister node with DS18B20</text>
-<text x="124.46" y="-76.2" size="2.54" layer="94" font="vector" ratio="15">Jon Sowman 04/17</text>
 </plain>
 <instances>
@@
 <instance part="GND7" gate="1" x="54.61" y="39.37" rot="R90"/>
 <instance part="C3" gate="G$1" x="149.86" y="-39.37"/>
+<instance part="SUPPLY6" gate="G$1" x="129.54" y="0"/>
 </instances>
 <busses>
@@
 </segment>
 <segment>
-<pinref part="R4" gate="G$1" pin="2"/>
-<wire x1="129.54" y1="-2.54" x2="129.54" y2="0" width="0.1524" layer="91"/>
-<label x="129.54" y="0" size="1.27" layer="95" font="vector" xref="yes"/>
-</segment>
-<segment>
 <pinref part="SUPPLY2" gate="G$1" pin="VCC"/>
 <wire x1="73.66" y1="2.54" x2="73.66" y2="0" width="0.1524" layer="91"/>
@@
 <pinref part="TC1" gate="A" pin="VCC"/>
 <pinref part="SUPPLY4" gate="G$1" pin="VCC"/>
+</segment>
+<segment>
+<pinref part="R4" gate="G$1" pin="2"/>
+<pinref part="SUPPLY6" gate="G$1" pin="VCC"/>
+<wire x1="129.54" y1="0" x2="129.54" y2="-2.54" width="0.1524" layer="91"/>
 </segment>
 </net>
@@
 <pinref part="U$1" gate="G$1" pin="PA9"/>
 <wire x1="209.55" y1="-27.94" x2="210.82" y2="-27.94" width="0.1524" layer="91"/>
-</segment>
-<segment>
+<label x="210.82" y="-27.94" size="1.27" layer="95" xref="yes"/>
+</segment>
+<segment>

Commit message: dumped some things on the pcb 12
Parts:
- removed TP4, TP5, TP6, TP7: TEST-POINT3, SparkFun-Passives:TEST-POINT3
Connections:
- net MISO: now also U$1.PA6; no longer TP6.1
- net MOSI: now also U$1.PA7; no longer TP5.1
- net RFM_SS: now also U$1.PA4; no longer TP4.1
- net SCK: now also U$1.PA5; no longer TP7.1
Changed lines of the file:
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@@
 <setting verticaltext="up"/>
 </settings>
-<grid distance="0.1" unitdist="inch" unit="inch" style="lines" multiple="1" display="no" altdistance="0.01" altunitdist="inch" altunit="inch"/>
+<grid distance="0.05" unitdist="inch" unit="inch" style="lines" multiple="1" display="no" altdistance="0.01" altunitdist="inch" altunit="inch"/>
 <layers>
 <layer number="1" name="Top" color="4" fill="1" visible="no" active="no"/>
@@
 <part name="R4" library="rcl" deviceset="R-EU_" device="R0603"/>
 <part name="TP1" library="SparkFun-Passives" deviceset="TEST-POINT" device="3"/>
-<part name="TP4" library="SparkFun-Passives" deviceset="TEST-POINT" device="3"/>
-<part name="TP5" library="SparkFun-Passives" deviceset="TEST-POINT" device="3"/>
-<part name="TP6" library="SparkFun-Passives" deviceset="TEST-POINT" device="3"/>
-<part name="TP7" library="SparkFun-Passives" deviceset="TEST-POINT" device="3"/>
 <part name="D2" library="SparkFun-LED" deviceset="WS2812B" device="" value="WS2812B"/>
 <part name="L1" library="passives-7351" deviceset="INDUCTOR" device="0603-N" value="4.7u"/>
@@
 <instance part="R4" gate="G$1" x="129.54" y="-7.62" rot="R90"/>
 <instance part="TP1" gate="G$1" x="134.62" y="48.26"/>
-<instance part="TP4" gate="G$1" x="200.66" y="50.8" smashed="yes">
-<attribute name="NAME" x="198.12" y="53.34" size="1.778" layer="95"/>
-</instance>
-<instance part="TP5" gate="G$1" x="200.66" y="45.72" smashed="yes">
-<attribute name="NAME" x="198.12" y="48.26" size="1.778" layer="95"/>
-</instance>
-<instance part="TP6" gate="G$1" x="200.66" y="40.64" smashed="yes">
-<attribute name="NAME" x="198.12" y="43.18" size="1.778" layer="95"/>
-</instance>
-<instance part="TP7" gate="G$1" x="200.66" y="35.56" smashed="yes">
-<attribute name="NAME" x="198.12" y="38.1" size="1.778" layer="95"/>
-</instance>
 <instance part="D2" gate="G$1" x="91.44" y="-5.08"/>
 <instance part="L1" gate="G$1" x="91.44" y="60.96"/>
@@
 <wire x1="190.5" y1="38.1" x2="200.66" y2="38.1" width="0.1524" layer="91"/>
 <label x="205.74" y="38.1" size="1.27" layer="95" font="vector" xref="yes"/>
-<pinref part="TP6" gate="G$1" pin="1"/>
 <wire x1="200.66" y1="38.1" x2="205.74" y2="38.1" width="0.1524" layer="91"/>
-<wire x1="200.66" y1="40.64" x2="200.66" y2="38.1" width="0.1524" layer="91"/>
-<junction x="200.66" y="38.1"/>
+</segment>
+<segment>
+<pinref part="U$1" gate="G$1" pin="PA6"/>
+<wire x1="209.55" y1="-20.32" x2="210.82" y2="-20.32" width="0.1524" layer="91"/>
+<label x="210.82" y="-20.32" size="1.27" layer="95" xref="yes"/>
 </segment>
 </net>
@@
 <wire x1="190.5" y1="43.18" x2="200.66" y2="43.18" width="0.1524" layer="91"/>
 <label x="205.74" y="43.18" size="1.27" layer="95" font="vector" xref="yes"/>
-<pinref part="TP5" gate="G$1" pin="1"/>
 <wire x1="200.66" y1="43.18" x2="205.74" y2="43.18" width="0.1524" layer="91"/>
-<wire x1="200.66" y1="45.72" x2="200.66" y2="43.18" width="0.1524" layer="91"/>
-<junction x="200.66" y="43.18"/>
+</segment>
+<segment>
+<pinref part="U$1" gate="G$1" pin="PA7"/>
+<wire x1="209.55" y1="-22.86" x2="210.82" y2="-22.86" width="0.1524" layer="91"/>
+<label x="210.82" y="-22.86" size="1.27" layer="95" xref="yes"/>
 </segment>
 </net>
@@
 <wire x1="190.5" y1="48.26" x2="200.66" y2="48.26" width="0.1524" layer="91"/>
 <label x="205.74" y="48.26" size="1.27" layer="95" font="vector" xref="yes"/>
-<pinref part="TP4" gate="G$1" pin="1"/>
 <wire x1="200.66" y1="48.26" x2="205.74" y2="48.26" width="0.1524" layer="91"/>
-<wire x1="200.66" y1="50.8" x2="200.66" y2="48.26" width="0.1524" layer="91"/>
-<junction x="200.66" y="48.26"/>
 </segment>
 <segment>
@@
 <label x="129.54" y="-15.24" size="1.27" layer="95" font="vector" xref="yes"/>
 </segment>
+<segment>
+<pinref part="U$1" gate="G$1" pin="PA4"/>
+<wire x1="209.55" y1="-15.24" x2="210.82" y2="-15.24" width="0.1524" layer="91"/>
+<label x="210.82" y="-15.24" size="1.27" layer="95" xref="yes"/>
+</segment>
 </net>
 <net name="N$3" class="0">
@@
 <wire x1="190.5" y1="33.02" x2="200.66" y2="33.02" width="0.1524" layer="91"/>
 <label x="205.74" y="33.02" size="1.27" layer="95" font="vector" xref="yes"/>
-<pinref part="TP7" gate="G$1" pin="1"/>
 <wire x1="200.66" y1="33.02" x2="205.74" y2="33.02" width="0.1524" layer="91"/>
-<wire x1="200.66" y1="35.56" x2="200.66" y2="33.02" width="0.1524" layer="91"/>
-<junction x="200.66" y="33.02"/>
-</segment>
-</net>
+</segment>
+<segment>
+<pinref part="U$1" gate="G$1" pin="PA5"/>
+<wire x1="209.55" y1="-17.78" x2="210.82" y2="-17.78" width="0.1524" layer="91"/>
+<label x="210.82" y="-17.78" size="1.27" layer="95" xref="yes"/>
+</segment>
+</net>

Commit message: commiting work on rgb-node
Parts:
- removed L1: 4.7u, passives-7351:INDUCTOR0603-N
- added C4: 10uF, SparkFun-Capacitors:10UF-POLAR-RADIAL-2.5MM-25V-20%
- added L2: 3.3µH/±20%/450mA, SparkFun-Coils:INDUCTOR-0805-3.3UH
Connections:
- new net VIB_SW: C4.+, U$1.PA0
- net GND: now also C4.-
- net N$1: now also L2.2; no longer L1.P$2
- net VBATT: now also L2.1; no longer L1.P$1
Other:
- note added: "Not a cap. Vibration switch."
Changed lines of the file:
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@@
 <?xml version="1.0" encoding="utf-8"?>
 <!DOCTYPE eagle SYSTEM "eagle.dtd">
-<eagle version="7.6.0">
+<eagle version="7.7.0">
 <drawing>
 <settings>
@@
 <part name="TP1" library="SparkFun-Passives" deviceset="TEST-POINT" device="3"/>
 <part name="D2" library="SparkFun-LED" deviceset="WS2812B" device="" value="WS2812B"/>
-<part name="L1" library="passives-7351" deviceset="INDUCTOR" device="0603-N" value="4.7u"/>
 <part name="BAT2" library="SparkFun" deviceset="BATTERY" device="AA"/>
 <part name="SUPPLY2" library="SparkFun-Aesthetics" deviceset="VCC" device=""/>
@@
 <part name="C3" library="passives-7351" deviceset="CAPACITOR" device="0603-N" value="100n"/>
 <part name="SUPPLY6" library="SparkFun-Aesthetics" deviceset="VCC" device=""/>
+<part name="C4" library="SparkFun-Capacitors" deviceset="10UF-POLAR" device="-RADIAL-2.5MM-25V-20%" value="10uF"/>
+<part name="GND8" library="SparkFun-Aesthetics" deviceset="GND" device=""/>
+<part name="L2" library="SparkFun-Coils" deviceset="INDUCTOR" device="-0805-3.3UH" value="3.3µH/±20%/450mA"/>
 </parts>
 <sheets>
 <sheet>
 <plain>
+<text x="78.74" y="-30.48" size="1.27" layer="91">Not a cap. Vibration switch.</text>
 </plain>
 <instances>
@@
 <instance part="TP1" gate="G$1" x="134.62" y="48.26"/>
 <instance part="D2" gate="G$1" x="91.44" y="-5.08"/>
-<instance part="L1" gate="G$1" x="91.44" y="60.96"/>
 <instance part="BAT2" gate="G$1" x="-27.94" y="48.26" rot="R270"/>
 <instance part="SUPPLY2" gate="G$1" x="73.66" y="2.54"/>
@@
 <instance part="C3" gate="G$1" x="149.86" y="-39.37"/>
 <instance part="SUPPLY6" gate="G$1" x="129.54" y="0"/>
+<instance part="C4" gate="G$1" x="99.06" y="-38.1"/>
+<instance part="GND8" gate="1" x="99.06" y="-45.72"/>
+<instance part="L2" gate="G$1" x="91.44" y="60.96" rot="R90"/>
 </instances>
 <busses>
@@
 <pinref part="GND7" gate="1" pin="GND"/>
 </segment>
+<segment>
+<pinref part="C4" gate="G$1" pin="-"/>
+<pinref part="GND8" gate="1" pin="GND"/>
+</segment>
 </net>
 <net name="VCC" class="0">
@@
 <wire x1="96.52" y1="60.96" x2="101.6" y2="60.96" width="0.1524" layer="91"/>
 <wire x1="101.6" y1="60.96" x2="101.6" y2="58.42" width="0.1524" layer="91"/>
-<pinref part="L1" gate="G$1" pin="P$2"/>
+<pinref part="L2" gate="G$1" pin="2"/>
 </segment>
 </net>
@@
 <segment>
 <wire x1="86.36" y1="60.96" x2="83.82" y2="60.96" width="0.1524" layer="91"/>
-<wire x1="83.82" y1="60.96" x2="83.82" y2="53.34" width="0.1524" layer="91"/>
+<wire x1="83.82" y1="60.96" x2="83.82" y2="48.26" width="0.1524" layer="91"/>
 <pinref part="U2" gate="G$1" pin="VIN"/>
-<wire x1="83.82" y1="53.34" x2="83.82" y2="48.26" width="0.1524" layer="91"/>
 <wire x1="83.82" y1="48.26" x2="86.36" y2="48.26" width="0.1524" layer="91"/>
 <label x="83.82" y="55.88" size="1.27" layer="95" font="vector" rot="R180" xref="yes"/>
@@
 <junction x="83.82" y="48.26"/>
 <pinref part="C2" gate="G$1" pin="1"/>
-<pinref part="L1" gate="G$1" pin="P$1"/>
 <pinref part="U2" gate="G$1" pin="EN"/>
 <wire x1="83.82" y1="43.18" x2="83.82" y2="35.56" width="0.1524" layer="91"/>
 <wire x1="86.36" y1="43.18" x2="83.82" y2="43.18" width="0.1524" layer="91"/>
 <junction x="83.82" y="43.18"/>
+<pinref part="L2" gate="G$1" pin="1"/>
 </segment>
 </net>
@@
 </segment>
 </net>
+<net name="VIB_SW" class="0">
+<segment>
+<pinref part="C4" gate="G$1" pin="+"/>
+<wire x1="99.06" y1="-35.56" x2="99.06" y2="-33.02" width="0.1524" layer="91"/>
+<wire x1="99.06" y1="-33.02" x2="101.6" y2="-33.02" width="0.1524" layer="91"/>
+<label x="101.6" y="-33.02" size="1.27" layer="95" xref="yes"/>
+</segment>
+<segment>
+<pinref part="U$1" gate="G$1" pin="PA0"/>
+<wire x1="209.55" y1="-5.08" x2="210.82" y2="-5.08" width="0.1524" layer="91"/>
+<label x="210.82" y="-5.08" size="1.27" layer="95" xref="yes"/>
+</segment>
+</net>
